File: tcrt5000/tcrt5000.kicad_pcb (KiCad board)
At the start: 2 copper layers, 17.1 x 12.1 mm, 7 parts, among them Q1 BC817, U1 TCRT5000, X1 Conn_01x03_Male

Commit message: Update
Other:
- board text added: "tnt23 2020"
Changed lines of the file:
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@@
   (general
     (thickness 1.6)
-    (drawings 4)
+    (drawings 5)
     (tracks 22)
     (zones 0)
@@
   )
   (setup
-    (last_trace_width 0.5)
+    (last_trace_width 0.25)
     (user_trace_width 0.3)
     (user_trace_width 0.5)
@@
     (visible_elements FFFFFF7F)
     (pcbplotparams
-      (layerselection 0x010fc_ffffffff)
+      (layerselection 0x010f0_ffffffff)
       (usegerberextensions false)
       (usegerberattributes false)
@@
       (psnegative false)
       (psa4output false)
-      (plotreference true)
-      (plotvalue true)
+      (plotreference false)
+      (plotvalue false)
       (plotinvisibletext false)
       (padsonsilk false)
@@
       (outputformat 1)
       (mirror false)
-      (drillshape 1)
+      (drillshape 0)
       (scaleselection 1)
-      (outputdirectory ""))
+      (outputdirectory "gerber/"))
   )
   (net 0 "")
@@
     (descr "Through hole straight pin header, 1x03, 2.54mm pitch, single row")
     (tags "Through hole pin header THT 1x03 2.54mm single row")
-    (fp_text reference X1 (at 0 -2.33) (layer F.SilkS)
+    (fp_text reference X1 (at 1.27 -1.905) (layer F.SilkS)
       (effects (font (size 1 1) (thickness 0.15)))
     )
@@
     (tags SOT-23)
     (attr smd)
-    (fp_text reference Q1 (at 0 2.5) (layer B.SilkS)
+    (fp_text reference Q1 (at -2.54 -1.27) (layer B.SilkS)
       (effects (font (size 1 1) (thickness 0.15)) (justify mirror))
     )
@@
   (module tcrt5000:TCRT500 (layer F.Cu)
     (at 132.29 87.63)
-    (fp_text reference U1 (at 0 -4.445) (layer F.SilkS)
+    (fp_text reference U1 (at 6.14 0) (layer F.SilkS)
       (effects (font (size 1 1) (thickness 0.15)))
     )
@@
     (pad "" np_thru_hole circle (at -4.65 2.54) (size 1 1) (drill 1) (layers *.Cu *.Mask))
   )
+  (gr_text "tnt23 2020" (at 132.08 92.71) (layer F.SilkS)
+    (effects (font (size 1 1) (thickness 0.15)))
+  )
   (gr_line (start 139.7 95.25) (end 139.7 83.185) (layer Edge.Cuts) (width 0.05))

Commit message: Mask updated
Routing:
- net /OUT: track 15.3 -> 14.6 mm
Other:
- board size 17.1 x 12.1 mm -> 16.5 x 12.1 mm
Changed lines of the file:
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@@
-(kicad_pcb (version 20171130) (host pcbnew 5.1.5-52549c5~84~ubuntu18.04.1)
+(kicad_pcb (version 20171130) (host pcbnew "(5.1.5)-2")
   (general
     (thickness 1.6)
-    (drawings 5)
+    (drawings 8)
     (tracks 22)
     (zones 0)
@@
     (solder_mask_min_width 0.25)
     (aux_axis_origin 0 0)
-    (visible_elements FFFFFF7F)
+    (visible_elements 7FFFFFFF)
     (pcbplotparams
       (layerselection 0x010f0_ffffffff)
@@
     (pad "" np_thru_hole circle (at -4.65 2.54) (size 1 1) (drill 1) (layers *.Cu *.Mask))
   )
+  (gr_poly (pts (xy 127.635 94.615) (xy 133.35 94.615) (xy 134.62 93.345) (xy 139.065 93.345) (xy 139.065 95.25) (xy 122.555 95.25) (xy 122.555 93.345) (xy 126.365 93.345)) (layer B.Mask) (width 0.1))
+  (gr_poly (pts (xy 139.065 85.09) (xy 122.555 85.09) (xy 122.555 83.185) (xy 139.065 83.185)) (layer B.Mask) (width 0.1))
+  (gr_line (start 137.16 83.185) (end 139.065 85.09) (layer Edge.Cuts) (width 0.05))
   (gr_text "tnt23 2020" (at 132.08 92.71) (layer F.SilkS)
     (effects (font (size 1 1) (thickness 0.15)))
   )
-  (gr_line (start 139.7 95.25) (end 139.7 83.185) (layer Edge.Cuts) (width 0.05))
-  (gr_line (start 122.555 95.25) (end 139.7 95.25) (layer Edge.Cuts) (width 0.05))
+  (gr_line (start 139.065 95.25) (end 139.065 85.09) (layer Edge.Cuts) (width 0.05))
+  (gr_line (start 122.555 95.25) (end 139.065 95.25) (layer Edge.Cuts) (width 0.05))
   (gr_line (start 122.555 83.185) (end 122.555 95.25) (layer Edge.Cuts) (width 0.05))
-  (gr_line (start 139.7 83.185) (end 122.555 83.185) (layer Edge.Cuts) (width 0.05))
+  (gr_line (start 137.16 83.185) (end 122.555 83.185) (layer Edge.Cuts) (width 0.05))
   (segment (start 135.6025 92.3775) (end 134.985 91.76) (width 0.5) (layer B.Cu) (net 1))
   (segment (start 137.16 92.3775) (end 135.6025 92.3775) (width 0.5) (layer B.Cu) (net 1))
@@
   (segment (start 124.7925 88.5675) (end 124.46 88.9) (width 0.5) (layer B.Cu) (net 5))
   (segment (start 127 88.5675) (end 124.7925 88.5675) (width 0.5) (layer B.Cu) (net 5))
+  (segment (start 126.365 90.805) (end 124.46 88.9) (width 0.5) (layer B.Cu) (net 5))
+  (segment (start 132.985 92.71) (end 132.935 92.71) (width 0.5) (layer B.Cu) (net 5))
+  (segment (start 126.365 92.075) (end 126.365 90.805) (width 0.5) (layer B.Cu) (net 5))
+  (segment (start 131.665 93.98) (end 128.27 93.98) (width 0.5) (layer B.Cu) (net 5))
   (segment (start 132.935 92.71) (end 131.665 93.98) (width 0.5) (layer B.Cu) (net 5))
-  (segment (start 132.985 92.71) (end 132.935 92.71) (width 0.5) (layer B.Cu) (net 5))
-  (segment (start 131.665 93.98) (end 127 93.98) (width 0.5) (layer B.Cu) (net 5))
-  (segment (start 127 93.98) (end 126.365 93.345) (width 0.5) (layer B.Cu) (net 5))
-  (segment (start 126.365 90.805) (end 124.46 88.9) (width 0.5) (layer B.Cu) (net 5))
-  (segment (start 126.365 93.345) (end 126.365 90.805) (width 0.5) (layer B.Cu) (net 5))
+  (segment (start 128.27 93.98) (end 126.365 92.075) (width 0.5) (layer B.Cu) (net 5))
   (segment (start 135.04 86.36) (end 133.77 87.63) (width 0.5) (layer B.Cu) (net 6))
   (segment (start 130.81 87.63) (end 129.54 86.36) (width 0.5) (layer B.Cu) (net 6))
@@
     (polygon
       (pts
-        (xy 139.7 95.25) (xy 120.65 95.25) (xy 120.65 83.185) (xy 139.7 83.185)
+        (xy 139.065 85.09) (xy 139.065 95.25) (xy 122.555 95.25) (xy 122.555 83.185) (xy 137.16 83.185)
       )
     )
