File: tcrt5000/tcrt5000.kicad_pcb (KiCad board)
At the start: 2 copper layers, 16.5 x 12.1 mm, 7 parts, among them Q1 BC817, U1 TCRT5000, X1 Conn_01x03_Male

Commit message: Gerbers done
Parts:
- added REF**: Gauge_50mm_Type2_SilkScreenTop, Measurement_Scales:Gauge_50mm_Type2_SilkScreenTop, F.Cu at (123.2, 95.2)
- moved R4 0.64 mm to (127.6, 87.6)
- moved X1 0.64 mm to (125.1, 86.4)
Routing:
- net /OUT: track 14.6 -> 13.9 mm
Other:
- board size 16.5 x 12.1 mm -> 15.9 x 12.1 mm
