File: DCC++ Shield/dccshield/dccshield.sch (KiCad schematic (older format))
At the start: 15 parts, among them J1 Conn_01x06, Q1 BTN8982TA, Q2 BTN8982TA, U1 74HC04, U2 A4953_LJ

Commit message: Up
Parts:
- added U?: 74HC04, Housings_SOIC:SOIC-14_3.9x8.7mm_Pitch1.27mm, symbol 74xx:74HC04
- R? (x2): value 510R -> 1K
Connections:
- net labels added: DCC_SIGNAL_MAIN, DCC_SIGNAL_PROG, ENABLE_MAIN
- wire segments 53 -> 54
Other:
- moved on the sheet: A1
Changed lines of the file:
@@
 $EndDescr
-$Comp
-L MCU_Module:Arduino_UNO_R3 A1
-U 1 1 5E38E585
-P 3850 4500
-F 0 "A1" H 3850 5950 50  0000 C CNN
-F 1 "Arduino_UNO_R3" H 3850 5875 50  0000 C CNN
-F 2 "Modules:Arduino_UNO_R3_WithMountingHoles" H 3850 5800 50  0000 C CIN
-F 3 "https://www.arduino.cc/en/Main/arduinoBoardUno" H 3850 4500 50  0001 C CNN
-	1    3850 4500
-	1    0    0    -1
-$EndComp
 $Comp
 L Power_Management:BTN8982TA Q1
@@
 	1    0    0    -1
 $EndComp
-Wire Wire Line
-	4050 3500 4050 3350
-Wire Wire Line
-	4050 3350 4500 3350
-Text GLabel 5000 3350 2    50   Output ~ 0
+Text GLabel 3000 3250 2    50   Output ~ 0
 +5V
 $Comp
@@
 Wire Wire Line
 	6750 2300 7200 2300
-Wire Wire Line
-	6750 3250 6500 3250
 Connection ~ 6750 3250
-Wire Wire Line
-	6675 3750 6500 3750
 Connection ~ 6675 3750
 Wire Wire Line
@@
 Connection ~ 6125 5300
 Wire Wire Line
-	6125 5300 5500 5300
+	6125 5300 4500 5300
 Text GLabel 7850 5600 0    50   Input ~ 0
 +5V
@@
 	1    0    0    -1
 $EndComp
+Wire Wire Line
+	8750 5500 9750 5500
+Wire Wire Line
+	9750 5500 9750 6250
+Wire Wire Line
+	9750 6250 6000 6250
+Connection ~ 8750 5500
+Wire Wire Line
+	2500 4200 2500 3250
+Wire Wire Line
+	2500 3250 3000 3250
+$Comp
+L power:GND #PWR?
+U 1 1 5E3CD4ED
+P 3300 2000
+F 0 "#PWR?" H 3300 1750 50  0001 C CNN
+F 1 "GND" H 3305 1827 50  0001 C CNN
+F 2 "" H 3300 2000 50  0001 C CNN
+F 3 "" H 3300 2000 50  0001 C CNN
+	1    3300 2000
+	1    0    0    -1
+$EndComp
+Text GLabel 3500 1000 2    50   Output ~ 0
++5V
+Wire Wire Line
+	3500 1000 3300 1000
+Text Notes 9250 5450 0    50   ~ 0
++/- 500mV ?
+Text Notes 9775 5725 0    50   ~ 0
+0R25 for Vref=5V and Imax=2A
+$Comp
+L Bridges:R R?
+U 1 1 5E3D5889
+P 7200 2850
+F 0 "R?" H 7400 2825 50  0000 R CNN
+F 1 "1K" H 7450 2900 50  0000 R CNN
+F 2 "Resistors_SMD:R_0805" V 7130 2850 50  0001 C CNN
+F 3 "" H 7200 2850 50  0001 C CNN
+	1    7200 2850
+	-1   0    0    1
+$EndComp
+$Comp
+L power:GND #PWR?
+U 1 1 5E3D6EA9
+P 7200 3000
+F 0 "#PWR?" H 7200 2750 50  0001 C CNN
+F 1 "GND" H 7205 2827 50  0001 C CNN
+F 2 "" H 7200 3000 50  0001 C CNN
+F 3 "" H 7200 3000 50  0001 C CNN
+	1    7200 3000
+	1    0    0    -1
+$EndComp
+$Comp
+L Bridges:R R?
+U 1 1 5E3D732F
+P 9275 2850
+F 0 "R?" H 9205 2804 50  0000 R CNN
+F 1 "1K" H 9205 2895 50  0000 R CNN
+F 2 "Resistors_SMD:R_0805" V 9205 2850 50  0001 C CNN
+F 3 "" H 9275 2850 50  0001 C CNN
+	1    9275 2850
+	-1   0    0    1
+$EndComp
+$Comp
+L power:GND #PWR?
+U 1 1 5E3D7339
+P 9275 3000
+F 0 "#PWR?" H 9275 2750 50  0001 C CNN
+F 1 "GND" H 9280 2827 50  0001 C CNN
+F 2 "" H 9275 3000 50  0001 C CNN
+F 3 "" H 9275 3000 50  0001 C CNN
+	1    9275 3000
+	1    0    0    -1
+$EndComp
+$Comp
+L Bridges:R R?
+U 1 1 5E3D8B55
+P 6950 4300
+F 0 "R?" H 6880 4254 50  0000 R CNN
+F 1 "TBD" H 6880 4345 50  0000 R CNN
+F 2 "Resistors_SMD:R_0805" V 6880 4300 50  0001 C CNN
+F 3 "" H 6950 4300 50  0001 C CNN
+	1    6950 4300
+	-1   0    0    1
+$EndComp
+$Comp
+L power:GND #PWR?
+U 1 1 5E3D8B5F
+P 6950 4450
+F 0 "#PWR?" H 6950 4200 50  0001 C CNN
+F 1 "GND" H 6955 4277 50  0001 C CNN
+F 2 "" H 6950 4450 50  0001 C CNN
+F 3 "" H 6950 4450 50  0001 C CNN
+	1    6950 4450
+	1    0    0    -1
+$EndComp
+Wire Wire Line
+	7200 2600 6950 2600
+Wire Wire Line
+	6950 2600 6950 4075
+Wire Wire Line
+	6950 4075 9925 4075
+Wire Wire Line
+	9925 4075 9925 2600
+Wire Wire Line
+	9925 2600 9275 2600
+Connection ~ 6950 4075
+Wire Wire Line
+	6950 4075 6950 4150
+$Comp
+L 74xx:74HC04 U?
+U 3 1 5E3E9EA5
+P 5300 3250
+F 0 "U?" H 5300 3600 50  0000 C CNN
+F 1 "74HC04" H 5300 3525 50  0000 C CNN
+F 2 "Housings_SOIC:SOIC-14_3.9x8.7mm_Pitch1.27mm" H 5300 3000 50  0000 C CNN
+F 3 "https://assets.nexperia.com/documents/data-sheet/74HC_HCT04.pdf" H 5300 3250 50  0001 C CNN
+	3    5300 3250
+	1    0    0    -1
+$EndComp
+Wire Wire Line
+	5000 3250 4500 3250
+Text Label 4500 3250 0    50   ~ 0
+ENABLE_MAIN
+Connection ~ 2500 3250
+$Comp
+L power:GND #PWR?
+U 1 1 5E3CCF82
+P 2250 6925
+F 0 "#PWR?" H 2250 6675 50  0001 C CNN
+F 1 "GND" H 2255 6752 50  0001 C CNN
+F 2 "" H 2250 6925 50  0001 C CNN
+F 3 "" H 2250 6925 50  0001 C CNN
+	1    2250 6925
+	1    0    0    -1
+$EndComp
+$Comp
+L power:GND #PWR?
+U 1 1 5E3CBEAB
+P 1950 5500
+F 0 "#PWR?" H 1950 5250 50  0001 C CNN
+F 1 "GND" H 1955 5327 50  0001 C CNN
+F 2 "" H 1950 5500 50  0001 C CNN
+F 3 "" H 1950 5500 50  0001 C CNN
+	1    1950 5500
+	1    0    0    -1
+$EndComp
+$Comp
+L power:GND #PWR?
+U 1 1 5E3CBCC4
+P 1850 5500
+F 0 "#PWR?" H 1850 5250 50  0001 C CNN
+F 1 "GND" H 1855 5327 50  0001 C CNN
+F 2 "" H 1850 5500 50  0001 C CNN
+F 3 "" H 1850 5500 50  0001 C CNN
+	1    1850 5500
+	1    0    0    -1
+$EndComp
+$Comp
+L power:GND #PWR?
+U 1 1 5E3CB802
+P 1750 5500
+F 0 "#PWR?" H 1750 5250 50  0001 C CNN
+F 1 "GND" H 1755 5327 50  0001 C CNN
+F 2 "" H 1750 5500 50  0001 C CNN
+F 3 "" H 1750 5500 50  0001 C CNN
+	1    1750 5500
+	1    0    0    -1
+$EndComp
+Wire Wire Line
+	2350 4200 2500 4200
 $Comp
 L Amplifier_Operational:LM358 U?
@@
 $EndComp
 Wire Wire Line
-	8750 5500 9750 5500
-Wire Wire Line
-	9750 5500 9750 6250
-Wire Wire Line
-	9750 6250 6000 6250
-Connection ~ 8750 5500
-Wire Wire Line
-	4350 4300 4500 4300
-Wire Wire Line
-	4500 4300 4500 3350
-Connection ~ 4500 3350
-Wire Wire Line
-	4500 3350 5000 3350
-$Comp
-L power:GND #PWR?
-U 1 1 5E3CB802
-P 3750 5600
-F 0 "#PWR?" H 3750 5350 50  0001 C CNN
-F 1 "GND" H 3755 5427 50  0001 C CNN
-F 2 "" H 3750 5600 50  0001 C CNN
-F 3 "" H 3750 5600 50  0001 C CNN
-	1    3750 5600
-	1    0    0    -1
-$EndComp
-$Comp
-L power:GND #PWR?
-U 1 1 5E3CBCC4
-P 3850 5600
-F 0 "#PWR?" H 3850 5350 50  0001 C CNN
-F 1 "GND" H 3855 5427 50  0001 C CNN
-F 2 "" H 3850 5600 50  0001 C CNN
-F 3 "" H 3850 5600 50  0001 C CNN
-	1    3850 5600
-	1    0    0    -1
-$EndComp
-$Comp
-L power:GND #PWR?
-U 1 1 5E3CBEAB
-P 3950 5600
-F 0 "#PWR?" H 3950 5350 50  0001 C CNN
-F 1 "GND" H 3955 5427 50  0001 C CNN
-F 2 "" H 3950 5600 50  0001 C CNN
-F 3 "" H 3950 5600 50  0001 C CNN
-	1    3950 5600
-	1    0    0    -1
-$EndComp
-$Comp
-L power:GND #PWR?
-U 1 1 5E3CCF82
-P 2250 6925
-F 0 "#PWR?" H 2250 6675 50  0001 C CNN
-F 1 "GND" H 2255 6752 50  0001 C CNN
-F 2 "" H 2250 6925 50  0001 C CNN
-F 3 "" H 2250 6925 50  0001 C CNN
-	1    2250 6925
-	1    0    0    -1
-$EndComp
-$Comp
-L power:GND #PWR?
-U 1 1 5E3CD4ED
-P 3300 2000
-F 0 "#PWR?" H 3300 1750 50  0001 C CNN
-F 1 "GND" H 3305 1827 50  0001 C CNN
-F 2 "" H 3300 2000 50  0001 C CNN
-F 3 "" H 3300 2000 50  0001 C CNN
-	1    3300 2000
-	1    0    0    -1
-$EndComp
-Text GLabel 3500 1000 2    50   Output ~ 0
-+5V
-Wire Wire Line
-	3500 1000 3300 1000
-Text Notes 9250 5450 0    50   ~ 0
-+/- 500mV ?
-Text Notes 9775 5725 0    50   ~ 0
-0R25 for Vref=5V and Imax=2A
+	2050 3250 2500 3250
+Wire Wire Line
+	2050 3400 2050 3250
+$Comp
+L MCU_Module:Arduino_UNO_R3 A1
+U 1 1 5E38E585
+P 1850 4400
+F 0 "A1" H 1850 5850 50  0000 C CNN
+F 1 "Arduino_UNO_R3" H 1850 5775 50  0000 C CNN
+F 2 "Modules:Arduino_UNO_R3_WithMountingHoles" H 1850 5700 50  0000 C CIN
+F 3 "https://www.arduino.cc/en/Main/arduinoBoardUno" H 1850 4400 50  0001 C CNN
+	1    1850 4400
+	1    0    0    -1
+$EndComp
+Text Label 4500 3750 0    50   ~ 0
+DCC_SIGNAL_MAIN
+Text Label 4500 5300 0    50   ~ 0
+DCC_SIGNAL_PROG
+Wire Wire Line
+	6675 3750 6500 3750
+Wire Wire Line
+	6200 3750 4500 3750
+Wire Wire Line
+	6750 3250 6500 3250
+Wire Wire Line
+	5600 3250 6200 3250
 $Comp
 L Bridges:R R?
@@
 	0    1    1    0
 $EndComp
-$Comp
-L Bridges:R R?
-U 1 1 5E3D5889
-P 7200 2850
-F 0 "R?" H 7400 2825 50  0000 R CNN
-F 1 "510R" H 7450 2900 50  0000 R CNN
-F 2 "Resistors_SMD:R_0805" V 7130 2850 50  0001 C CNN
-F 3 "" H 7200 2850 50  0001 C CNN
-	1    7200 2850
-	-1   0    0    1
-$EndComp
-$Comp
-L power:GND #PWR?
-U 1 1 5E3D6EA9
-P 7200 3000
-F 0 "#PWR?" H 7200 2750 50  0001 C CNN
-F 1 "GND" H 7205 2827 50  0001 C CNN
-F 2 "" H 7200 3000 50  0001 C CNN
-F 3 "" H 7200 3000 50  0001 C CNN
-	1    7200 3000
-	1    0    0    -1
-$EndComp
-$Comp
-L Bridges:R R?
-U 1 1 5E3D732F
-P 9275 2850
-F 0 "R?" H 9205 2804 50  0000 R CNN
-F 1 "510R" H 9205 2895 50  0000 R CNN
-F 2 "Resistors_SMD:R_0805" V 9205 2850 50  0001 C CNN
-F 3 "" H 9275 2850 50  0001 C CNN
-	1    9275 2850
-	-1   0    0    1
-$EndComp
-$Comp
-L power:GND #PWR?
-U 1 1 5E3D7339
-P 9275 3000
-F 0 "#PWR?" H 9275 2750 50  0001 C CNN
-F 1 "GND" H 9280 2827 50  0001 C CNN
-F 2 "" H 9275 3000 50  0001 C CNN
-F 3 "" H 9275 3000 50  0001 C CNN
-	1    9275 3000
-	1    0    0    -1
-$EndComp
-$Comp
-L Bridges:R R?
-U 1 1 5E3D8B55
-P 6950 4300
-F 0 "R?" H 6880 4254 50  0000 R CNN
-F 1 "TBD" H 6880 4345 50  0000 R CNN
-F 2 "Resistors_SMD:R_0805" V 6880 4300 50  0001 C CNN
-F 3 "" H 6950 4300 50  0001 C CNN
-	1    6950 4300
-	-1   0    0    1
-$EndComp
-$Comp
-L power:GND #PWR?
-U 1 1 5E3D8B5F
-P 6950 4450
-F 0 "#PWR?" H 6950 4200 50  0001 C CNN
-F 1 "GND" H 6955 4277 50  0001 C CNN
-F 2 "" H 6950 4450 50  0001 C CNN
-F 3 "" H 6950 4450 50  0001 C CNN
-	1    6950 4450
-	1    0    0    -1
-$EndComp
-Wire Wire Line
-	7200 2600 6950 2600
-Wire Wire Line
-	6950 2600 6950 4075
-Wire Wire Line
-	6950 4075 9925 4075
-Wire Wire Line
-	9925 4075 9925 2600
-Wire Wire Line
-	9925 2600 9275 2600
-Connection ~ 6950 4075
-Wire Wire Line
-	6950 4075 6950 4150
-Wire Wire Line
-	6200 3250 5750 3250
-Wire Wire Line
-	6200 3750 5750 3750
 $EndSCHEMATC

Commit message: Update
Parts:
- added R10, R3, R8: 10K, Resistors_SMD:R_0805, symbol Bridges:R
- added R11, R12: DNF, Resistors_SMD:R_0805, symbol Bridges:R
- added R6, R9: 1K, Resistors_SMD:R_0805, symbol Bridges:R
- U3: renamed from U?; footprint (none) -> Housings_SOIC:SOIC-8_3.9x4.9mm_Pitch1.27mm
- gave numbers to parts that had none: 7
- renumbered Rs to Rs1
Connections:
- net DCC_SIGNAL_MAIN: now also A1.25 (D10), R12.2
- net DCC_SIGNAL_PROG: now also A1.20 (D5), R11.2, R3.2; no longer U1.3, U2.3 (IN1)
- net ENABLE_MAIN: now also A1.18 (D3), R1.2; no longer U1.5
- net GND: now also J1.2 (Pin_2), R6.1, R9.1; no longer J1.4 (Pin_4)
- net MAIN1: now also J1.3 (Pin_3); no longer J1.1 (Pin_1)
- net MAIN2: now also J1.4 (Pin_4); no longer J1.2 (Pin_2)
- net PROG1: now also U2.8 (OUT2); no longer U2.6 (OUT1)
- net PROG2: now also U2.6 (OUT1); no longer U2.8 (OUT2)
- net VCC: now also J1.1 (Pin_1); no longer J1.3 (Pin_3)
- net A1: now reaches A1.10 (A1)
- net A1: now also U3.7, R8.1
- net at A1.17 (D2): now also R11.1
- net at A1.27 (D12): now also R12.1
- net A0: now reaches A1.9 (A0)
- net A0: now also U3.1, R10.1
- net at Q1.2 (IN), R2.1: now also U1.5; no longer U1.1
- net at Q1.3 (INH), Q2.3 (INH): now also U1.2; no longer R1.1
- net at Q1.6 (IS), Q2.6 (IS), R7.2: now also U3.3 (+)
- net at Q2.2 (IN): now also U1.6; no longer U1.2
- net at Rs1.1, U2.7 (LSS): now also U3.5 (+)
- net at U3.2 (-): now also R10.2, R9.2
- net at U3.6 (-): now also R6.2, R8.2
- new net: R3.1, U1.3, U2.3 (IN1)
- new net: R1.1, U1.1
Other:
- note added: "ENABLE PROG ???"
- note added: "TBD"
- moved on the sheet: A1, J1, Q1, Q2, R1, R2, R4, R5, R7, Rs1, U1A, U1B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
