File: DCC++ Shield/dccshield/dccshield.sch (KiCad schematic (older format))
At the start: 28 parts, among them J1 Conn_01x06, Q1 BTN8982TA, Q2 BTN8982TA, U1 74HC04, U2 A4953_LJ, U3 LM358

Commit message: PCB update
Connections:
- net DCC_SIGNAL_MAIN: now also Q1.2 (IN), U1.5; no longer A1.25 (D10)
- new net: A1.25 (D10), R2.1
Other:
- moved on the sheet: R2
Changed lines of the file:
@@
 Text Label 2750 5050 0    50   ~ 0
 DCC_SIGNAL_PROG
-Wire Wire Line
-	5175 3475 4375 3475
-Wire Wire Line
-	4075 3475 3375 3475
 $Comp
 L Bridges:R R2
 U 1 1 5E3D389B
-P 4225 3475
-F 0 "R2" V 4018 3475 50  0000 C CNN
-F 1 "10K" V 4109 3475 50  0000 C CNN
-F 2 "Resistors_SMD:R_0805" V 4155 3475 50  0001 C CNN
-F 3 "" H 4225 3475 50  0001 C CNN
-	1    4225 3475
+P 1950 2450
+F 0 "R2" V 1743 2450 50  0000 C CNN
+F 1 "10K" V 1834 2450 50  0000 C CNN
+F 2 "Resistors_SMD:R_0805" V 1880 2450 50  0001 C CNN
+F 3 "" H 1950 2450 50  0001 C CNN
+	1    1950 2450
 	0    1    1    0
 $EndComp
@@
 U 1 1 5E36F49C
 P 1925 2650
-F 0 "R12" V 1718 2650 50  0000 C CNN
-F 1 "DNF" V 1809 2650 50  0000 C CNN
+F 0 "R12" V 2025 2650 50  0000 C CNN
+F 1 "DNF" V 2100 2650 50  0000 C CNN
 F 2 "Resistors_SMD:R_0805" V 1855 2650 50  0001 C CNN
 F 3 "" H 1925 2650 50  0001 C CNN
@@
 Wire Wire Line
 	1725 2650 1725 2450
-Connection ~ 1725 2450
-Wire Wire Line
-	1725 2450 2225 2450
 Wire Wire Line
 	2225 1650 1700 1650
@@
 Wire Wire Line
 	6750 2700 6750 1900
+Wire Wire Line
+	3375 3475 5175 3475
+Wire Wire Line
+	1800 2450 1725 2450
+Connection ~ 1725 2450
+Wire Wire Line
+	2100 2450 2225 2450
 $EndSCHEMATC
