File: DCC++ Shield/dccshield/dccshield.sch (KiCad schematic (older format))
At the start: 29 parts, among them J1 Conn_01x06, Q1 BTN8982TA, Q2 BTN8982TA, U1 74HC04, U2 A4953_LJ, U3 LM358

Commit message: up
Parts:
- gave numbers to parts that had none: 1
Other:
- note added: "Resistanse is futile. Inductance is not."
Changed lines of the file:
@@
 	2100 2450 2225 2450
 $Comp
-L Device:Ferrite_Bead_Small FB?
+L Device:Ferrite_Bead_Small FB1
 U 1 1 5E3E685D
 P 3400 4025
-F 0 "FB?" V 3073 4025 50  0000 C CNN
+F 0 "FB1" V 3073 4025 50  0000 C CNN
 F 1 "Ferrite_Bead_Small" V 3164 4025 50  0000 C CNN
 F 2 "Inductors_SMD:L_0805_HandSoldering" V 3255 4025 50  0000 C CNN
@@
 $EndComp
 $Comp
-L power:GND #PWR?
+L power:GND #PWR0122
 U 1 1 5E3E774A
 P 3300 4025
-F 0 "#PWR?" H 3300 3775 50  0001 C CNN
+F 0 "#PWR0122" H 3300 3775 50  0001 C CNN
 F 1 "GND" H 3305 3852 50  0001 C CNN
 F 2 "" H 3300 4025 50  0001 C CNN
@@
 $EndComp
 $Comp
-L power:GND #PWR?
+L power:GND #PWR0123
 U 1 1 5E3E7E28
 P 3500 4025
-F 0 "#PWR?" H 3500 3775 50  0001 C CNN
+F 0 "#PWR0123" H 3500 3775 50  0001 C CNN
 F 1 "GND" H 3505 3852 50  0001 C CNN
 F 2 "" H 3500 4025 50  0001 C CNN
@@
 	1    0    0    -1
 $EndComp
+Text Notes 2775 4225 0    50   ~ 0
+Resistanse is futile. Inductance is not.
 $EndSCHEMATC

Commit message: Gerbers, docs
Other:
- note added: "For MEGA"
- note added: "For UNO"
Changed lines of the file:
@@
 encoding utf-8
 Sheet 1 1
-Title ""
-Date ""
-Rev ""
-Comp ""
+Title "DCC++ Shield"
+Date "2020-01-30"
+Rev "0.1"
+Comp "Tim Tashpulatov"
 Comment1 ""
 Comment2 ""
@@
 U 2 1 5E3A88F7
 P 4800 5450
-F 0 "U1" H 4800 5857 50  0000 C CNN
-F 1 "74HC04" H 4800 5766 50  0000 C CNN
-F 2 "Housings_SOIC:SOIC-14_3.9x8.7mm_Pitch1.27mm" H 4800 5675 50  0000 C CNN
+F 0 "U1" H 4800 5750 50  0000 C CNN
+F 1 "74HC04" H 4850 5650 50  0000 C CNN
+F 2 "Housings_SOIC:SOIC-14_3.9x8.7mm_Pitch1.27mm" H 4350 5200 50  0000 C CNN
 F 3 "https://assets.nexperia.com/documents/data-sheet/74HC_HCT04.pdf" H 4800 5450 50  0001 C CNN
 	2    4800 5450
@@
 F 0 "U3" H 8550 5717 50  0000 C CNN
 F 1 "LM358" H 8550 5626 50  0000 C CNN
-F 2 "Housings_SOIC:SOIC-8_3.9x4.9mm_Pitch1.27mm" H 9525 5575 50  0000 C CNN
+F 2 "Housings_SOIC:SOIC-8_3.9x4.9mm_Pitch1.27mm" H 9525 5525 50  0000 C CNN
 F 3 "http://www.ti.com/lit/ds/symlink/lm2904-n.pdf" H 8550 5350 50  0001 C CNN
 	2    8550 5350
@@
 Text Notes 7500 5200 0    50   ~ 0
 +/- 500mV ?
-Text Notes 7300 4925 0    50   ~ 0
+Text Notes 6850 6025 0    50   ~ 0
 0R25 for Vref=5V and Imax=2A
 $Comp
@@
 Wire Wire Line
 	3550 5050 2750 5050
-Text Notes 4250 4675 0    50   ~ 0
+Text Notes 1500 4625 0    50   ~ 0
 ENABLE PROG ???
 Text Label 3225 2050 0    50   ~ 0
@@
 U 1 1 5E35866A
 P 9600 4325
-F 0 "R10" V 9393 4325 50  0000 C CNN
-F 1 "10K" V 9484 4325 50  0000 C CNN
+F 0 "R10" V 9500 4325 50  0000 C CNN
+F 1 "10K" V 9700 4325 50  0000 C CNN
 F 2 "Resistors_SMD:R_0805" V 9530 4325 50  0001 C CNN
 F 3 "" H 9600 4325 50  0001 C CNN
@@
 P 9250 4550
 F 0 "R9" H 9125 4525 50  0000 C CNN
-F 1 "1K" H 9100 4625 50  0000 C CNN
+F 1 "1K" H 9125 4625 50  0000 C CNN
 F 2 "Resistors_SMD:R_0805" V 9180 4550 50  0001 C CNN
 F 3 "" H 9250 4550 50  0001 C CNN
@@
 Wire Wire Line
 	9850 4325 9850 3900
-Text Notes 9550 4575 0    50   ~ 0
+Text Notes 9800 4750 0    50   ~ 0
 TBD
 Wire Wire Line
@@
 F 0 "C3" H 5840 5591 50  0000 L CNN
 F 1 "100nF" H 5840 5500 50  0000 L CNN
-F 2 "Capacitors_SMD:C_0805" H 4825 5400 50  0000 L CNN
+F 2 "Capacitors_SMD:C_0805" H 5300 5400 50  0000 L CNN
 F 3 "" H 5725 5500 50  0001 C CNN
 	1    5725 5500
@@
 Text Notes 2775 4225 0    50   ~ 0
 Resistanse is futile. Inductance is not.
+Text Notes 1450 2050 0    50   ~ 0
+For UNO
+Text Notes 1425 1525 0    50   ~ 0
+For MEGA
+Text Notes 1425 2850 0    50   ~ 0
+For MEGA
+Text Notes 1525 2300 0    50   ~ 0
+For UNO
 $EndSCHEMATC

Commit message: Update and gerbers
Parts:
- removed R11, R12: DNF, Resistors_SMD:R_0805, symbol Bridges:R
- added JP1, JP2: MAIN UNO/MEGA, Pin_Headers:Pin_Header_Straight_1x03_Pitch2.54mm, symbol Jumper:Jumper_3_Open
Connections:
- net DCC_SIGNAL_MAIN: now also R2.1, JP2.2 (C); no longer Q1.2 (IN), R2.2, U1.5
- net DCC_SIGNAL_PROG: now also JP1.2 (C); no longer A1.20 (D5)
- net at A1.27 (D12): now also JP2.3 (B)
- net at A1.17 (D2): now also JP1.1 (A)
- net at A1.25 (D10): now also JP2.1 (A); no longer R2.1
- new net: A1.20 (D5), JP1.3 (B)
- new net: Q1.2 (IN), R2.2, U1.5
Other:
- moved on the sheet: R2, R3
Changed lines of the file:
@@
 Connection ~ 4375 5050
 Wire Wire Line
-	4375 5050 3850 5050
+	4375 5050 4350 5050
 Text GLabel 5650 5350 0    50   Input ~ 0
 +5V
@@
 	1    0    0    -1
 $EndComp
-Text Label 3375 3475 0    50   ~ 0
+Text Label 3400 3475 0    50   ~ 0
 DCC_SIGNAL_MAIN
-Text Label 2750 5050 0    50   ~ 0
+Text Label 3250 5050 0    50   ~ 0
 DCC_SIGNAL_PROG
 $Comp
 L Bridges:R R2
 U 1 1 5E3D389B
-P 1950 2450
-F 0 "R2" V 1743 2450 50  0000 C CNN
-F 1 "10K" V 1834 2450 50  0000 C CNN
-F 2 "Resistors_SMD:R_0805" V 1880 2450 50  0001 C CNN
-F 3 "" H 1950 2450 50  0001 C CNN
-	1    1950 2450
-	0    1    1    0
+P 4225 3475
+F 0 "R2" V 4018 3475 50  0000 C CNN
+F 1 "10K" V 4109 3475 50  0000 C CNN
+F 2 "Resistors_SMD:R_0805" V 4155 3475 50  0001 C CNN
+F 3 "" H 4225 3475 50  0001 C CNN
+	1    4225 3475
+	0    -1   -1   0
 $EndComp
 $Comp
@@
 L Bridges:R R3
 U 1 1 5E34FD15
-P 3700 5050
-F 0 "R3" V 3493 5050 50  0000 C CNN
-F 1 "10K" V 3584 5050 50  0000 C CNN
-F 2 "Resistors_SMD:R_0805" V 3630 5050 50  0001 C CNN
-F 3 "" H 3700 5050 50  0001 C CNN
-	1    3700 5050
+P 4200 5050
+F 0 "R3" V 3993 5050 50  0000 C CNN
+F 1 "10K" V 4084 5050 50  0000 C CNN
+F 2 "Resistors_SMD:R_0805" V 4130 5050 50  0001 C CNN
+F 3 "" H 4200 5050 50  0001 C CNN
+	1    4200 5050
 	0    1    1    0
 $EndComp
 Wire Wire Line
-	3550 5050 2750 5050
+	4050 5050 3250 5050
 Text Notes 1500 4625 0    50   ~ 0
 ENABLE PROG ???
@@
 Text Label 2225 1750 2    50   ~ 0
 ENABLE_MAIN
-Text Label 1625 2450 2    50   ~ 0
+Text Label 625  2575 2    50   ~ 0
 DCC_SIGNAL_MAIN
-Text Label 1275 1950 2    50   ~ 0
+Text Label 550  1800 2    50   ~ 0
 DCC_SIGNAL_PROG
-Wire Wire Line
-	2225 2650 2075 2650
-$Comp
-L Bridges:R R12
-U 1 1 5E36F49C
-P 1925 2650
-F 0 "R12" V 2025 2650 50  0000 C CNN
-F 1 "DNF" V 2100 2650 50  0000 C CNN
-F 2 "Resistors_SMD:R_0805" V 1855 2650 50  0001 C CNN
-F 3 "" H 1925 2650 50  0001 C CNN
-	1    1925 2650
-	0    1    1    0
-$EndComp
-Wire Wire Line
-	1625 2450 1725 2450
-Wire Wire Line
-	1775 2650 1725 2650
-Wire Wire Line
-	1725 2650 1725 2450
-Wire Wire Line
-	2225 1650 1700 1650
-$Comp
-L Bridges:R R11
-U 1 1 5E3736A4
-P 1550 1650
-F 0 "R11" V 1343 1650 50  0000 C CNN
-F 1 "DNF" V 1434 1650 50  0000 C CNN
-F 2 "Resistors_SMD:R_0805" V 1480 1650 50  0001 C CNN
-F 3 "" H 1550 1650 50  0001 C CNN
-	1    1550 1650
-	0    1    -1   0
-$EndComp
-Wire Wire Line
-	1400 1650 1350 1650
-Wire Wire Line
-	1350 1650 1350 1950
-Wire Wire Line
-	2225 1950 1350 1950
-Connection ~ 1350 1950
-Wire Wire Line
-	1350 1950 1275 1950
 $Comp
 L Bridges:C C1
@@
 	6750 2700 6750 1900
 Wire Wire Line
-	3375 3475 5175 3475
-Wire Wire Line
-	1800 2450 1725 2450
-Connection ~ 1725 2450
-Wire Wire Line
-	2100 2450 2225 2450
+	4375 3475 5175 3475
 $Comp
 L Device:Ferrite_Bead_Small FB1
@@
 Text Notes 2775 4225 0    50   ~ 0
 Resistanse is futile. Inductance is not.
-Text Notes 1450 2050 0    50   ~ 0
+Text Notes 950  2150 0    50   ~ 0
 For UNO
-Text Notes 1425 1525 0    50   ~ 0
+Text Notes 900  1500 0    50   ~ 0
 For MEGA
-Text Notes 1425 2850 0    50   ~ 0
+Text Notes 1000 2950 0    50   ~ 0
 For MEGA
-Text Notes 1525 2300 0    50   ~ 0
+Text Notes 975  2300 0    50   ~ 0
 For UNO
+Wire Wire Line
+	775  2575 625  2575
+$Comp
+L Jumper:Jumper_3_Open JP2
+U 1 1 5E5C8CD0
+P 925 2575
+F 0 "JP2" V 834 2662 50  0000 L CNN
+F 1 "MAIN UNO/MEGA" V 925 2662 50  0000 L CNN
+F 2 "Pin_Headers:Pin_Header_Straight_1x03_Pitch2.54mm" V 1016 2662 50  0000 L CNN
+F 3 "~" H 925 2575 50  0001 C CNN
+	1    925  2575
+	0    1    1    0
+$EndComp
+Wire Wire Line
+	925  2325 1400 2325
+Wire Wire Line
+	1400 2325 1400 2450
+Wire Wire Line
+	1400 2450 2225 2450
+Wire Wire Line
+	925  2825 1400 2825
+Wire Wire Line
+	1400 2825 1400 2650
+Wire Wire Line
+	1400 2650 2225 2650
+Wire Wire Line
+	4075 3475 3400 3475
+Wire Wire Line
+	1275 1950 2225 1950
+$Comp
+L Jumper:Jumper_3_Open JP1
+U 1 1 5E5E66B9
+P 925 1800
+F 0 "JP1" V 834 1887 50  0000 L CNN
+F 1 "MAIN UNO/MEGA" V 925 1887 50  0000 L CNN
+F 2 "Pin_Headers:Pin_Header_Straight_1x03_Pitch2.54mm" V 1016 1887 50  0000 L CNN
+F 3 "~" H 925 1800 50  0001 C CNN
+	1    925  1800
+	0    1    1    0
+$EndComp
+Wire Wire Line
+	925  2050 1275 2050
+Wire Wire Line
+	1275 2050 1275 1950
+Wire Wire Line
+	925  1550 1275 1550
+Wire Wire Line
+	1275 1550 1275 1650
+Wire Wire Line
+	1275 1650 2225 1650
+Wire Wire Line
+	775  1800 550  1800
 $EndSCHEMATC
