File: DCC++ Shield/dccshield/_autosave-dccshield.sch (KiCad schematic (older format))
At the start: 28 parts, among them J1 Conn_01x06, Q1 BTN8982TA, Q2 BTN8982TA, U1 74HC04, U2 A4953_LJ, U3 LM358

Commit message: PCB update
Parts:
- gave numbers to parts that had none: 1
Changed lines of the file:
@@
 	8425 2325 8600 2325
 $Comp
-L Device:CP1 C?
+L Device:CP1 C6
 U 1 1 5E44E46C
 P 6750 1750
-F 0 "C?" H 6865 1841 50  0000 L CNN
+F 0 "C6" H 6865 1841 50  0000 L CNN
 F 1 "100uF 50V" H 6865 1750 50  0000 L CNN
 F 2 "Capacitors_SMD:CP_Elec_6.3x5.3" H 6800 2075 50  0000 L CNN
