File: DCC++ Shield/dccshield/_autosave-dccshield.kicad_pcb (KiCad board)
At the start: 2 copper layers, 57.2 x 53.3 mm, 29 parts, among them Q1 BTN8982TA, Q2 BTN8982TA, U1 74HC04, U2 A4953_LJ, U3 LM358, X1 Conn_01x06

Commit message: Gerbers, docs
Other:
- board text added: "DCC++ SHIELD v0.1"
- board text added: "tnt23 2020"
Changed lines of the file:
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@@
   (general
     (thickness 1.6)
-    (drawings 9)
+    (drawings 11)
     (tracks 269)
     (zones 0)
@@
     (tags "SOIC 1.27")
     (attr smd)
-    (fp_text reference U3 (at 0 -3.5) (layer F.SilkS)
+    (fp_text reference U3 (at 0 3.81) (layer F.SilkS)
       (effects (font (size 1 1) (thickness 0.15)))
     )
@@
     )
   )
+  (gr_text "tnt23 2020" (at 144.145 101.6 90) (layer F.SilkS)
+    (effects (font (size 1.5 1.5) (thickness 0.25)))
+  )
+  (gr_text "DCC++ SHIELD v0.1" (at 139.7 101.6 90) (layer F.SilkS)
+    (effects (font (size 2 2) (thickness 0.5)))
+  )
   (gr_line (start 190.5 78.74) (end 190.5 76.2) (layer Edge.Cuts) (width 0.05))
