File: DCC++ Shield/dccshield/dccshield.kicad_pcb (KiCad board)
At the start: 2 copper layers, 57.2 x 53.3 mm, 29 parts, among them Q1 BTN8982TA, Q2 BTN8982TA, U1 74HC04, U2 A4953_LJ, U3 LM358, X1 Conn_01x06

Commit message: Update and gerbers
Parts:
- removed R11, R12: DNF, Resistors_SMD:R_0805
- added JP1: MAIN UNO/MEGA, Pin_Headers:Pin_Header_Straight_1x03_Pitch2.54mm, F.Cu at (139.7, 106.7)
- added JP2: MAIN UNO/MEGA, Pin_Headers:Pin_Header_Straight_1x03_Pitch2.54mm, F.Cu at (139.7, 116.8)
- moved R2 29.2 mm to (139.7, 103.5), turned to 0 degrees
- moved R3 24.4 mm to (142.9, 110.5), turned to 90 degrees
- renumbered X1 to J1
Connections:
- A1 pad 20: /DCC_SIGNAL_PROG -> Net-(A1-Pad20)
- Q1 pad 2: /DCC_SIGNAL_MAIN -> Net-(Q1-Pad2)
- R2 pad 1: Net-(A1-Pad25) -> /DCC_SIGNAL_MAIN
- R2 pad 2: /DCC_SIGNAL_MAIN -> Net-(Q1-Pad2)
- U1 pad 5: /DCC_SIGNAL_MAIN -> Net-(Q1-Pad2)
Routing:
- net Net-(A1-Pad20): track 0.00 -> 44.0 mm
- net Net-(Q1-Pad2): track 0.00 -> 41.9 mm, vias 0 -> 3
- net Net-(A1-Pad17): track 18.9 -> 55.6 mm, vias 1 -> 2
- net /DCC_SIGNAL_MAIN: track 54.1 -> 18.2 mm, vias 3 -> 0
- net Net-(A1-Pad25): track 2.54 -> 25.5 mm
- net Net-(A1-Pad27): track 2.54 -> 21.3 mm
- net /DCC_SIGNAL_PROG: track 14.8 -> 3.31 mm
- net MAIN2: track 22.1 -> 10.9 mm
- net MAIN1: track 22.4 -> 11.5 mm
- net Net-(R3-Pad1): track 35.4 -> 37.4 mm
- net /ENABLE_MAIN: track 34.5 -> 33.0 mm
- net +5V: track 50.6 -> 51.4 mm
- net GND: vias 32 -> 41
- added copper zone on F.Cu, net MAIN1
- added copper zone on F.Cu, net MAIN2
Other:
- board text added: "+"
- board text added: "-"
- board text added: "DCC++ Shield 1.0 (c) 2020 tnt23"
- board text added: "JP1"
- board text added: "JP2"
- board text added: "M"
- board text added: "MEGA"
- board text added: "P"
- board text added: "UNO"
- board text added: "■"
