File: loco/loco/loco.sch (KiCad schematic (older format))
At the start: 1 part, among them U1 STM32F030F4Px

Commit message: Loco update
Parts:
- added D1: NSR2030, loco:NSR2030, symbol loco:NSR2030
- added U2: A4953_LJ, Package_SO:SOIC-8-1EP_3.9x4.9mm_P1.27mm_EP2.41x3.3mm, symbol Driver_Motor:A4953_LJ
Connections:
- net labels added: 27V, RAIL1, RAIL2
- wire segments 0 -> 9
Changed lines of the file:
@@
 $EndComp
 $Comp
-L power:GND #PWR?
+L power:GND #PWR0101
 U 1 1 5E6518CE
 P 5650 4300
-F 0 "#PWR?" H 5650 4050 50  0001 C CNN
+F 0 "#PWR0101" H 5650 4050 50  0001 C CNN
 F 1 "GND" H 5655 4127 50  0001 C CNN
 F 2 "" H 5650 4300 50  0001 C CNN
@@
 	1    0    0    -1
 $EndComp
+$Comp
+L loco:NSR2030 D1
+U 1 1 5E65250C
+P 2500 2350
+F 0 "D1" H 2500 2715 50  0000 C CNN
+F 1 "NSR2030" H 2500 2624 50  0000 C CNN
+F 2 "loco:NSR2030" H 2500 2533 50  0000 C CNN
+F 3 "" H 2500 2350 50  0001 C CNN
+	1    2500 2350
+	1    0    0    -1
+$EndComp
+Wire Wire Line
+	2750 2400 2900 2400
+Wire Wire Line
+	2900 2400 2900 2575
+Wire Wire Line
+	2900 2575 1975 2575
+Wire Wire Line
+	2250 2300 1975 2300
+Text GLabel 1975 2300 0    50   Input ~ 0
+RAIL1
+Text GLabel 1975 2575 0    50   Input ~ 0
+RAIL2
+$Comp
+L power:GND #PWR0102
+U 1 1 5E652E8A
+P 2875 2025
+F 0 "#PWR0102" H 2875 1775 50  0001 C CNN
+F 1 "GND" H 2880 1852 50  0001 C CNN
+F 2 "" H 2875 2025 50  0001 C CNN
+F 3 "" H 2875 2025 50  0001 C CNN
+	1    2875 2025
+	-1   0    0    1
+$EndComp
+Wire Wire Line
+	2875 2025 2875 2300
+Wire Wire Line
+	2875 2300 2750 2300
+Wire Wire Line
+	2250 2400 2175 2400
+Wire Wire Line
+	2175 2400 2175 2700
+Wire Wire Line
+	2175 2700 3175 2700
+$Comp
+L Driver_Motor:A4953_LJ U2
+U 1 1 5E653C2B
+P 3200 4325
+F 0 "U2" H 3200 4906 50  0000 C CNN
+F 1 "A4953_LJ" H 3200 4815 50  0000 C CNN
+F 2 "Package_SO:SOIC-8-1EP_3.9x4.9mm_P1.27mm_EP2.41x3.3mm" H 3200 3775 50  0001 C CNN
+F 3 "www.allegromicro.com/~/media/Files/Datasheets/A4952-3-Datasheet.ashx?la=en" H 2900 4675 50  0001 C CNN
+	1    3200 4325
+	1    0    0    -1
+$EndComp
+Text Label 2850 2700 0    50   ~ 0
+27V
 $EndSCHEMATC

Commit message: Update
Connections:
- net labels added: +3V3, BOOT0, IN1, IN2, M1, M2, NRST
- wire segments 9 -> 19
Changed lines of the file:
@@
 U 1 1 5E653C2B
 P 3200 4325
-F 0 "U2" H 3200 4906 50  0000 C CNN
-F 1 "A4953_LJ" H 3200 4815 50  0000 C CNN
+F 0 "U2" H 3400 4800 50  0000 C CNN
+F 1 "A4953_LJ" H 3425 4700 50  0000 C CNN
 F 2 "Package_SO:SOIC-8-1EP_3.9x4.9mm_P1.27mm_EP2.41x3.3mm" H 3200 3775 50  0001 C CNN
 F 3 "www.allegromicro.com/~/media/Files/Datasheets/A4952-3-Datasheet.ashx?la=en" H 2900 4675 50  0001 C CNN
@@
 Text Label 2850 2700 0    50   ~ 0
 27V
+Text Label 5150 3000 2    50   ~ 0
+NRST
+Text Label 5150 3200 2    50   ~ 0
+BOOT0
+Wire Wire Line
+	5650 2800 5650 2700
+Wire Wire Line
+	5750 2800 5750 2700
+Wire Wire Line
+	5750 2700 5650 2700
+Connection ~ 5650 2700
+Wire Wire Line
+	5650 2700 5650 2600
+Text Label 5650 2600 0    50   ~ 0
++3V3
+$Comp
+L power:GND #PWR?
+U 1 1 5E657AD9
+P 3200 4825
+F 0 "#PWR?" H 3200 4575 50  0001 C CNN
+F 1 "GND" H 3205 4652 50  0001 C CNN
+F 2 "" H 3200 4825 50  0001 C CNN
+F 3 "" H 3200 4825 50  0001 C CNN
+	1    3200 4825
+	1    0    0    -1
+$EndComp
+Wire Wire Line
+	3200 4725 3200 4775
+Wire Wire Line
+	3300 4725 3300 4775
+Wire Wire Line
+	3300 4775 3200 4775
+Connection ~ 3200 4775
+Wire Wire Line
+	3200 4775 3200 4825
+Wire Wire Line
+	3600 4125 3825 4125
+Wire Wire Line
+	3600 4225 3825 4225
+Text Label 3825 4125 0    50   ~ 0
+M1
+Text Label 3825 4225 0    50   ~ 0
+M2
+Text Label 2800 4125 2    50   ~ 0
+IN1
+Text Label 2800 4225 2    50   ~ 0
+IN2
+Text Label 3200 3925 2    50   ~ 0
+27V
 $EndSCHEMATC

Commit message: Up
Parts:
- added U3: TLV760, Package_TO_SOT_SMD:SOT-23, symbol loco:TLV760
Connections:
- wire segments 19 -> 24
Other:
- moved on the sheet: D1, U2
Changed lines of the file:
@@
 L loco:NSR2030 D1
 U 1 1 5E65250C
-P 2500 2350
-F 0 "D1" H 2500 2715 50  0000 C CNN
-F 1 "NSR2030" H 2500 2624 50  0000 C CNN
-F 2 "loco:NSR2030" H 2500 2533 50  0000 C CNN
-F 3 "" H 2500 2350 50  0001 C CNN
-	1    2500 2350
+P 2500 2250
+F 0 "D1" H 2500 2615 50  0000 C CNN
+F 1 "NSR2030" H 2500 2524 50  0000 C CNN
+F 2 "loco:NSR2030" H 2500 2433 50  0000 C CNN
+F 3 "" H 2500 2250 50  0001 C CNN
+	1    2500 2250
 	1    0    0    -1
 $EndComp
 Wire Wire Line
-	2750 2400 2900 2400
+	2750 2300 2900 2300
 Wire Wire Line
-	2900 2400 2900 2575
+	2900 2300 2900 2475
 Wire Wire Line
-	2900 2575 1975 2575
+	2900 2475 1975 2475
 Wire Wire Line
-	2250 2300 1975 2300
-Text GLabel 1975 2300 0    50   Input ~ 0
+	2250 2200 1975 2200
+Text GLabel 1975 2200 0    50   Input ~ 0
 RAIL1
-Text GLabel 1975 2575 0    50   Input ~ 0
+Text GLabel 1975 2475 0    50   Input ~ 0
 RAIL2
 $Comp
 L power:GND #PWR0102
 U 1 1 5E652E8A
-P 2875 2025
-F 0 "#PWR0102" H 2875 1775 50  0001 C CNN
-F 1 "GND" H 2880 1852 50  0001 C CNN
-F 2 "" H 2875 2025 50  0001 C CNN
-F 3 "" H 2875 2025 50  0001 C CNN
-	1    2875 2025
+P 2875 1925
+F 0 "#PWR0102" H 2875 1675 50  0001 C CNN
+F 1 "GND" H 2880 1752 50  0001 C CNN
+F 2 "" H 2875 1925 50  0001 C CNN
+F 3 "" H 2875 1925 50  0001 C CNN
+	1    2875 1925
 	-1   0    0    1
 $EndComp
 Wire Wire Line
-	2875 2025 2875 2300
+	2875 1925 2875 2200
 Wire Wire Line
-	2875 2300 2750 2300
+	2875 2200 2750 2200
 Wire Wire Line
-	2250 2400 2175 2400
+	2250 2300 2175 2300
 Wire Wire Line
-	2175 2400 2175 2700
+	2175 2300 2175 2600
 Wire Wire Line
-	2175 2700 3175 2700
+	2175 2600 3075 2600
 $Comp
 L Driver_Motor:A4953_LJ U2
 U 1 1 5E653C2B
-P 3200 4325
-F 0 "U2" H 3400 4800 50  0000 C CNN
-F 1 "A4953_LJ" H 3425 4700 50  0000 C CNN
-F 2 "Package_SO:SOIC-8-1EP_3.9x4.9mm_P1.27mm_EP2.41x3.3mm" H 3200 3775 50  0001 C CNN
-F 3 "www.allegromicro.com/~/media/Files/Datasheets/A4952-3-Datasheet.ashx?la=en" H 2900 4675 50  0001 C CNN
-	1    3200 4325
-	1    0    0    -1
+P 3075 4025
+F 0 "U2" H 3275 4500 50  0000 C CNN
+F 1 "A4953_LJ" H 3300 4400 50  0000 C CNN
+F 2 "Package_SO:SOIC-8-1EP_3.9x4.9mm_P1.27mm_EP2.41x3.3mm" H 3075 3475 50  0001 C CNN
+F 3 "www.allegromicro.com/~/media/Files/Datasheets/A4952-3-Datasheet.ashx?la=en" H 2775 4375 50  0001 C CNN
+	1    3075 4025
+	-1   0    0    -1
 $EndComp
-Text Label 2850 2700 0    50   ~ 0
+Text Label 2850 2600 0    50   ~ 0
 27V
 Text Label 5150 3000 2    50   ~ 0
@@
 +3V3
 $Comp
-L power:GND #PWR?
+L power:GND #PWR0103
 U 1 1 5E657AD9
-P 3200 4825
-F 0 "#PWR?" H 3200 4575 50  0001 C CNN
-F 1 "GND" H 3205 4652 50  0001 C CNN
-F 2 "" H 3200 4825 50  0001 C CNN
-F 3 "" H 3200 4825 50  0001 C CNN
-	1    3200 4825
+P 3075 4525
+F 0 "#PWR0103" H 3075 4275 50  0001 C CNN
+F 1 "GND" H 3080 4352 50  0001 C CNN
+F 2 "" H 3075 4525 50  0001 C CNN
+F 3 "" H 3075 4525 50  0001 C CNN
+	1    3075 4525
+	-1   0    0    -1
+$EndComp
+Wire Wire Line
+	3075 4425 3075 4475
+Wire Wire Line
+	2975 4425 2975 4475
+Wire Wire Line
+	2975 4475 3075 4475
+Connection ~ 3075 4475
+Wire Wire Line
+	3075 4475 3075 4525
+Wire Wire Line
+	2675 3825 2450 3825
+Wire Wire Line
+	2675 3925 2450 3925
+Text Label 2450 3825 2    50   ~ 0
+M1
+Text Label 2450 3925 2    50   ~ 0
+M2
+Text Label 3475 3825 0    50   ~ 0
+IN1
+Text Label 3475 3925 0    50   ~ 0
+IN2
+$Comp
+L loco:TLV760 U3
+U 1 1 5E653E6E
+P 3475 3100
+F 0 "U3" H 3653 3216 50  0000 L CNN
+F 1 "TLV760" H 3653 3125 50  0000 L CNN
+F 2 "Package_TO_SOT_SMD:SOT-23" H 3653 3034 50  0000 L CNN
+F 3 "" H 3475 3200 50  0001 C CNN
+	1    3475 3100
+	1    0    0    -1
+$EndComp
+$Comp
+L power:GND #PWR0104
+U 1 1 5E654599
+P 3475 3300
+F 0 "#PWR0104" H 3475 3050 50  0001 C CNN
+F 1 "GND" H 3480 3127 50  0001 C CNN
+F 2 "" H 3475 3300 50  0001 C CNN
+F 3 "" H 3475 3300 50  0001 C CNN
+	1    3475 3300
 	1    0    0    -1
 $EndComp
 Wire Wire Line
-	3200 4725 3200 4775
+	3375 2600 3375 2850
 Wire Wire Line
-	3300 4725 3300 4775
+	3575 2850 3575 2600
 Wire Wire Line
-	3300 4775 3200 4775
-Connection ~ 3200 4775
+	3575 2600 5650 2600
 Wire Wire Line
-	3200 4775 3200 4825
+	3075 3625 3075 2600
+Connection ~ 3075 2600
 Wire Wire Line
-	3600 4125 3825 4125
-Wire Wire Line
-	3600 4225 3825 4225
-Text Label 3825 4125 0    50   ~ 0
-M1
-Text Label 3825 4225 0    50   ~ 0
-M2
-Text Label 2800 4125 2    50   ~ 0
-IN1
-Text Label 2800 4225 2    50   ~ 0
-IN2
-Text Label 3200 3925 2    50   ~ 0
-27V
+	3075 2600 3375 2600
 $EndSCHEMATC

Commit message: Update
Parts:
- added C1, C2: C, Capacitor_SMD:C_0603_1608Metric, symbol Device:C
Connections:
- net labels added: SWCLK, SWDIO
- wire segments 24 -> 34
Changed lines of the file:
@@
 Wire Wire Line
 	2175 2300 2175 2600
-Wire Wire Line
-	2175 2600 3075 2600
 $Comp
 L Driver_Motor:A4953_LJ U2
@@
 	3575 2850 3575 2600
 Wire Wire Line
-	3575 2600 5650 2600
+	3575 2600 4350 2600
 Wire Wire Line
 	3075 3625 3075 2600
@@
 Wire Wire Line
 	3075 2600 3375 2600
+$Comp
+L Device:C C1
+U 1 1 5E65CF36
+P 2550 2875
+F 0 "C1" H 2665 2921 50  0000 L CNN
+F 1 "C" H 2665 2830 50  0000 L CNN
+F 2 "Capacitor_SMD:C_0603_1608Metric" H 2588 2725 50  0001 C CNN
+F 3 "~" H 2550 2875 50  0001 C CNN
+	1    2550 2875
+	1    0    0    -1
+$EndComp
+Wire Wire Line
+	2550 2725 2550 2600
+Wire Wire Line
+	2175 2600 2550 2600
+Connection ~ 2550 2600
+Wire Wire Line
+	2550 2600 3075 2600
+$Comp
+L power:GND #PWR0105
+U 1 1 5E65D4B8
+P 2550 3025
+F 0 "#PWR0105" H 2550 2775 50  0001 C CNN
+F 1 "GND" H 2555 2852 50  0001 C CNN
+F 2 "" H 2550 3025 50  0001 C CNN
+F 3 "" H 2550 3025 50  0001 C CNN
+	1    2550 3025
+	1    0    0    -1
+$EndComp
+$Comp
+L Device:C C2
+U 1 1 5E65E01F
+P 4350 2825
+F 0 "C2" H 4465 2871 50  0000 L CNN
+F 1 "C" H 4465 2780 50  0000 L CNN
+F 2 "Capacitor_SMD:C_0603_1608Metric" H 4388 2675 50  0001 C CNN
+F 3 "~" H 4350 2825 50  0001 C CNN
+	1    4350 2825
+	1    0    0    -1
+$EndComp
+$Comp
+L power:GND #PWR0106
+U 1 1 5E65E029
+P 4350 2975
+F 0 "#PWR0106" H 4350 2725 50  0001 C CNN
+F 1 "GND" H 4355 2802 50  0001 C CNN
+F 2 "" H 4350 2975 50  0001 C CNN
+F 3 "" H 4350 2975 50  0001 C CNN
+	1    4350 2975
+	1    0    0    -1
+$EndComp
+Wire Wire Line
+	4350 2675 4350 2600
+Connection ~ 4350 2600
+Wire Wire Line
+	4350 2600 5650 2600
+Wire Wire Line
+	6150 4000 6550 4000
+Wire Wire Line
+	6550 4000 6550 4325
+Connection ~ 6550 4000
+Wire Wire Line
+	6550 4000 6750 4000
+Text Label 6550 4325 0    50   ~ 0
+SWDIO
+Wire Wire Line
+	6150 4100 6325 4100
+Wire Wire Line
+	6325 4100 6325 4425
+Connection ~ 6325 4100
+Wire Wire Line
+	6325 4100 6750 4100
+Text Label 6325 4425 0    50   ~ 0
+SWCLK
 $EndSCHEMATC

Commit message: Update
Parts:
- added R1: TBD, Resistor_SMD:R_0603_1608Metric, symbol Device:R
Connections:
- net labels added: ADC_IN0, ADC_IN1, ADC_IN3, ADC_IN4, LSS, TIM14_CH1, TIM3_CH1, TIM3_CH2, VREF
- net labels removed: IN1, IN2
- wire segments 34 -> 48
Other:
- note added: "TIM1_CH2"
- note added: "TIM1_CH3"
- note added: "TIM3_CH4, TIM14_CH1, TIM1_CH3"
Changed lines of the file:
@@
 Wire Wire Line
 	2675 3825 2450 3825
-Wire Wire Line
-	2675 3925 2450 3925
-Text Label 2450 3825 2    50   ~ 0
-M1
-Text Label 2450 3925 2    50   ~ 0
-M2
-Text Label 3475 3825 0    50   ~ 0
-IN1
-Text Label 3475 3925 0    50   ~ 0
-IN2
 $Comp
 L loco:TLV760 U3
@@
 Text Label 6325 4425 0    50   ~ 0
 SWCLK
+Text Label 6150 3000 0    50   ~ 0
+ADC_IN0
+Text Label 6150 3100 0    50   ~ 0
+ADC_IN1
+Text Label 6150 3200 0    50   ~ 0
+ADC_IN3
+Text Label 6150 3300 0    50   ~ 0
+ADC_IN4
+Text Notes 5050 4100 2    39   ~ 0
+TIM3_CH4, TIM14_CH1, TIM1_CH3
+Text Notes 6225 3800 0    39   ~ 0
+TIM1_CH2
+Text Notes 6225 3900 0    39   ~ 0
+TIM1_CH3
+Text Label 6500 3400 0    39   ~ 0
+TIM14_CH1
+Wire Wire Line
+	6150 3400 6900 3400
+Wire Wire Line
+	6900 3400 6900 2750
+$Comp
+L Device:R R1
+U 1 1 5E66806A
+P 6900 2600
+F 0 "R1" H 6970 2646 50  0000 L CNN
+F 1 "TBD" H 6970 2555 50  0000 L CNN
+F 2 "Resistor_SMD:R_0603_1608Metric" V 6830 2600 50  0001 C CNN
+F 3 "~" H 6900 2600 50  0001 C CNN
+	1    6900 2600
+	1    0    0    -1
+$EndComp
+Wire Wire Line
+	6900 2450 6900 2300
+Wire Wire Line
+	6900 2300 2900 2300
+Connection ~ 2900 2300
+Text GLabel 2450 3825 0    50   Output ~ 0
+M1
+Wire Wire Line
+	2675 3925 2450 3925
+Text GLabel 2450 3925 0    50   Output ~ 0
+M2
+Text Label 6225 3600 0    39   ~ 0
+TIM3_CH1
+Wire Wire Line
+	6150 3700 6900 3700
+Text Label 6225 3700 0    39   ~ 0
+TIM3_CH2
+Wire Wire Line
+	3675 3825 3675 4675
+Wire Wire Line
+	3675 4675 6900 4675
+Wire Wire Line
+	6900 4675 6900 3700
+Wire Wire Line
+	7000 3600 7000 4775
+Wire Wire Line
+	7000 4775 3750 4775
+Wire Wire Line
+	3750 4775 3750 3925
+Wire Wire Line
+	6150 3600 7000 3600
+Wire Wire Line
+	3750 3925 3475 3925
+Wire Wire Line
+	3675 3825 3475 3825
+Text Label 3475 4125 0    50   ~ 0
+VREF
+Text Label 2675 4025 2    50   ~ 0
+LSS
 $EndSCHEMATC

Commit message: Update
Parts:
- added C?: C, Capacitor_SMD:C_0603_1608Metric, symbol Device:C
Connections:
- net labels added: F1, F2, F3, F4, F5
- wire segments 48 -> 52
Other:
- moved on the sheet: R1
Changed lines of the file:
@@
 TIM14_CH1
 Wire Wire Line
-	6150 3400 6900 3400
+	6150 3400 6975 3400
 Wire Wire Line
-	6900 3400 6900 2750
+	6975 3400 6975 2750
 $Comp
 L Device:R R1
 U 1 1 5E66806A
-P 6900 2600
-F 0 "R1" H 6970 2646 50  0000 L CNN
-F 1 "TBD" H 6970 2555 50  0000 L CNN
-F 2 "Resistor_SMD:R_0603_1608Metric" V 6830 2600 50  0001 C CNN
-F 3 "~" H 6900 2600 50  0001 C CNN
-	1    6900 2600
+P 6975 2600
+F 0 "R1" H 7045 2646 50  0000 L CNN
+F 1 "TBD" H 7045 2555 50  0000 L CNN
+F 2 "Resistor_SMD:R_0603_1608Metric" V 6905 2600 50  0001 C CNN
+F 3 "~" H 6975 2600 50  0001 C CNN
+	1    6975 2600
 	1    0    0    -1
 $EndComp
 Wire Wire Line
-	6900 2450 6900 2300
+	6975 2450 6975 2300
 Wire Wire Line
-	6900 2300 2900 2300
+	6975 2300 2900 2300
 Connection ~ 2900 2300
 Text GLabel 2450 3825 0    50   Output ~ 0
@@
 Text Label 2675 4025 2    50   ~ 0
 LSS
+$Comp
+L Device:C C?
+U 1 1 5E687C29
+P 6600 2700
+F 0 "C?" H 6715 2746 50  0000 L CNN
+F 1 "C" H 6715 2655 50  0000 L CNN
+F 2 "Capacitor_SMD:C_0603_1608Metric" H 6638 2550 50  0001 C CNN
+F 3 "~" H 6600 2700 50  0001 C CNN
+	1    6600 2700
+	1    0    0    -1
+$EndComp
+$Comp
+L power:GND #PWR?
+U 1 1 5E687C33
+P 6600 2850
+F 0 "#PWR?" H 6600 2600 50  0001 C CNN
+F 1 "GND" H 6605 2677 50  0001 C CNN
+F 2 "" H 6600 2850 50  0001 C CNN
+F 3 "" H 6600 2850 50  0001 C CNN
+	1    6600 2850
+	1    0    0    -1
+$EndComp
+Wire Wire Line
+	6600 2550 6600 2400
+Wire Wire Line
+	6600 2400 6125 2400
+Wire Wire Line
+	6125 2400 6125 2700
+Wire Wire Line
+	6125 2700 5750 2700
+Connection ~ 5750 2700
+Text GLabel 8825 3600 2    50   Output ~ 0
+F1
+Text GLabel 8825 3725 2    50   Output ~ 0
+F2
+Text GLabel 8825 3850 2    50   Output ~ 0
+F3
+Text GLabel 8825 3975 2    50   Output ~ 0
+F4
+Text GLabel 8825 4100 2    50   Output ~ 0
+F5
 $EndSCHEMATC

Commit message: FR and RL
Parts:
- added C4: 100n, Capacitor_SMD:C_0603_1608Metric, symbol Device:C
- added Q1, Q2, Q3: FDC6561AN, Package_TO_SOT_SMD:SuperSOT-6, symbol loco:FDC6561AN
- added R2, R3: 10K, Resistor_SMD:R_0603_1608Metric, symbol Device:R
- added R4, R5, R6, R7, R8, R9: TBD, Resistor_SMD:R_0603_1608Metric, symbol Device:R
- gave numbers to parts that had none: 1
Connections:
- net labels added: FL, RL, _FL, _RL
- net labels removed: LSS, VREF
- wire segments 52 -> 89

Commit message: F1 and F2
Parts:
- added C5: C, Capacitor_SMD:C_0603_1608Metric, symbol Device:C
Connections:
- net labels added: _F1, _F2
- net labels removed: ADC_IN3, ADC_IN4
- wire segments 89 -> 92
Changed lines of the file:
@@
 	3575 2600 3975 2600
 Wire Wire Line
-	3075 3625 3075 2600
+	3075 3625 3075 2875
 Connection ~ 3075 2600
 Wire Wire Line
@@
 Text Label 6150 3100 0    50   ~ 0
 ADC_IN1
-Text Label 6150 3200 0    50   ~ 0
-ADC_IN3
-Text Label 6150 3300 0    50   ~ 0
-ADC_IN4
 Text Notes 4975 4100 2    39   ~ 0
 TIM3_CH4, TIM14_CH1, TIM1_CH3
@@
 Text Label 5150 4100 2    50   ~ 0
 _FL
+Text Label 8400 2800 0    50   ~ 0
+_F1
+Text Label 8400 3000 0    50   ~ 0
+_F2
+Text Label 6150 3200 0    50   ~ 0
+_F1
+Text Label 6150 3300 0    50   ~ 0
+_F2
+$Comp
+L Device:C C5
+U 1 1 5E6B1D41
+P 2900 3150
+F 0 "C5" H 3015 3196 50  0000 L CNN
+F 1 "C" H 3015 3105 50  0000 L CNN
+F 2 "Capacitor_SMD:C_0603_1608Metric" H 2938 3000 50  0001 C CNN
+F 3 "~" H 2900 3150 50  0001 C CNN
+	1    2900 3150
+	1    0    0    -1
+$EndComp
+Wire Wire Line
+	2900 3000 2900 2875
+$Comp
+L power:GND #PWR0115
+U 1 1 5E6B1D4C
+P 2900 3300
+F 0 "#PWR0115" H 2900 3050 50  0001 C CNN
+F 1 "GND" H 2905 3127 50  0001 C CNN
+F 2 "" H 2900 3300 50  0001 C CNN
+F 3 "" H 2900 3300 50  0001 C CNN
+	1    2900 3300
+	1    0    0    -1
+$EndComp
+Wire Wire Line
+	2900 2875 3075 2875
+Connection ~ 3075 2875
+Wire Wire Line
+	3075 2875 3075 2600
 $EndSCHEMATC
